Commit message: Add files via upload

File: wall_e_description/urdf/wall_e.xacro (robot description, xacro)
@@ -84,4 +84,24 @@
   </collision>
 </link>
+<link name="ydlidar_x4_1">
+  <inertial>
+    <origin xyz="-0.008294104236280672 -4.075333863429176e-08 0.03520110343257382" rpy="0 0 0"/>
+    <mass value="1.1515616542314233"/>
+    <inertia ixx="0.000489" iyy="0.000861" izz="0.000987" ixy="-0.0" iyz="0.0" ixz="-0.000148"/>
+  </inertial>
+  <visual>
+    <origin xyz="-0.032937 -0.040618 -0.336435" rpy="0 0 0"/>
+    <geometry>
+      <mesh filename="package://wall_e_description/meshes/ydlidar_x4_1.stl" scale="0.001 0.001 0.001"/>
+    </geometry>
+    <material name="steel_satin"/>
+  </visual>
+  <collision>
+    <origin xyz="-0.032937 -0.040618 -0.336435" rpy="0 0 0"/>
+    <geometry>
+      <mesh filename="package://wall_e_description/meshes/ydlidar_x4_1.stl" scale="0.001 0.001 0.001"/>
+    </geometry>
+  </collision>
+</link>
 <joint name="left_drive" type="continuous">
   <origin xyz="0.032937 -0.094382 0.054935" rpy="0 0 0"/>
@@ -101,3 +121,8 @@
   <child link="bin_1"/>
 </joint>
+<joint name="Rigid5" type="fixed">
+  <origin xyz="0.0 0.0 0.3" rpy="0 0 0"/>
+  <parent link="bin_1"/>
+  <child link="ydlidar_x4_1"/>
+</joint>
 </robot>

Commit message: Add files via upload

File: wall_e_description/urdf/wall_e.xacro (robot description, xacro)
@@ -24,5 +24,5 @@
   </collision>
 </link>
-<link name="right_wheel_1">
+<link name="right_wheel">
   <inertial>
     <origin xyz="-4.6659614505450975e-09 -0.010000040753338671 -3.879021768377067e-08" rpy="0 0 0"/>
@@ -44,5 +44,5 @@
   </collision>
 </link>
-<link name="left_wheel_1">
+<link name="left_wheel">
   <inertial>
     <origin xyz="-4.6659614505450975e-09 0.009999959246660972 -3.8790217787854075e-08" rpy="0 0 0"/>
@@ -64,5 +64,5 @@
   </collision>
 </link>
-<link name="bin_1">
+<link name="bin">
   <inertial>
     <origin xyz="0.022504658517767652 -0.00039207869774715576 0.17469334388419402" rpy="0 0 0"/>
@@ -84,5 +84,5 @@
   </collision>
 </link>
-<link name="ydlidar_x4_1">
+<link name="ydlidar_x4">
   <inertial>
     <origin xyz="-0.008294104236280672 -4.075333863429176e-08 0.03520110343257382" rpy="0 0 0"/>
@@ -91,5 +91,5 @@
   </inertial>
   <visual>
-    <origin xyz="-0.032937 -0.040618 -0.336435" rpy="0 0 0"/>
+    <origin xyz="-0.032937 -0.040618 -0.366435" rpy="0 0 0"/>
     <geometry>
       <mesh filename="package://wall_e_description/meshes/ydlidar_x4_1.stl" scale="0.001 0.001 0.001"/>
@@ -107,11 +107,11 @@
   <origin xyz="0.032937 -0.094382 0.054935" rpy="0 0 0"/>
   <parent link="base_link"/>
-  <child link="right_wheel_1"/>
-  <axis xyz="-0.0 -1.0 0.0"/>
+  <child link="left_wheel"/>
+  <axis xyz="-0.0 1.0 0.0"/>
 </joint>
 <joint name="right_drive" type="continuous">
   <origin xyz="0.032937 0.175618 0.054935" rpy="0 0 0"/>
   <parent link="base_link"/>
-  <child link="left_wheel_1"/>
+  <child link="right_wheel"/>
   <axis xyz="0.0 1.0 -0.0"/>
 </joint>
@@ -119,10 +119,10 @@
   <origin xyz="0.032937 0.040618 0.036435" rpy="0 0 0"/>
   <parent link="base_link"/>
-  <child link="bin_1"/>
+  <child link="bin"/>
 </joint>
 <joint name="Rigid5" type="fixed">
-  <origin xyz="0.0 0.0 0.3" rpy="0 0 0"/>
-  <parent link="bin_1"/>
-  <child link="ydlidar_x4_1"/>
+  <origin xyz="0.0 0.0 0.33" rpy="0 0 0"/>
+  <parent link="bin"/>
+  <child link="ydlidar_x4"/>
 </joint>
 </robot>

Commit message: Add files via upload

File: wall_e_description/urdf/wall_e.xacro (robot description, xacro)
@@ -6,5 +6,5 @@
 <link name="base_link">
   <inertial>
-    <origin xyz="0.032936995334038474 0.04061795924666118 0.042779283007869824" rpy="0 0 0"/>
+    <origin xyz="0.03306922009986352 0.04109957889568825 0.041731230355942464" rpy="0 0 0"/>
     <mass value="4.787456478250945"/>
     <inertia ixx="0.027048" iyy="0.030516" izz="0.054315" ixy="-0.0" iyz="0.0" ixz="-0.0"/>
@@ -24,52 +24,52 @@
   </collision>
 </link>
-<link name="right_wheel">
-  <inertial>
-    <origin xyz="-4.6659614505450975e-09 -0.010000040753338671 -3.879021768377067e-08" rpy="0 0 0"/>
+<link name="right_wheel_1">
+  <inertial>
+    <origin xyz="2.2009986355014943e-07 -0.010000421104311583 -9.144214505041326e-08" rpy="0 0 0"/>
+    <mass value="0.17676171065422966"/>
+    <inertia ixx="0.00014" iyy="0.000267" izz="0.00014" ixy="0.0" iyz="-0.0" ixz="-0.0"/>
+  </inertial>
+  <visual>
+    <origin xyz="-0.033069 0.0939 -0.053887" rpy="0 0 0"/>
+    <geometry>
+      <mesh filename="package://wall_e_description/meshes/right_wheel_1.stl" scale="0.001 0.001 0.001"/>
+    </geometry>
+    <material name="rubber_soft"/>
+  </visual>
+  <collision>
+    <origin xyz="-0.033069 0.0939 -0.053887" rpy="0 0 0"/>
+    <geometry>
+      <mesh filename="package://wall_e_description/meshes/right_wheel_1.stl" scale="0.001 0.001 0.001"/>
+    </geometry>
+  </collision>
+</link>
+<link name="left_wheel_1">
+  <inertial>
+    <origin xyz="2.2009986355014943e-07 0.009999578895688033 -9.144214514755777e-08" rpy="0 0 0"/>
     <mass value="0.17676171065422966"/>
     <inertia ixx="0.00014" iyy="0.000267" izz="0.00014" ixy="-0.0" iyz="0.0" ixz="-0.0"/>
   </inertial>
   <visual>
-    <origin xyz="-0.032937 0.094382 -0.054935" rpy="0 0 0"/>
-    <geometry>
-      <mesh filename="package://wall_e_description/meshes/right_wheel_1.stl" scale="0.001 0.001 0.001"/>
+    <origin xyz="-0.033069 -0.1761 -0.053887" rpy="0 0 0"/>
+    <geometry>
+      <mesh filename="package://wall_e_description/meshes/left_wheel_1.stl" scale="0.001 0.001 0.001"/>
     </geometry>
     <material name="rubber_soft"/>
   </visual>
   <collision>
-    <origin xyz="-0.032937 0.094382 -0.054935" rpy="0 0 0"/>
-    <geometry>
-      <mesh filename="package://wall_e_description/meshes/right_wheel_1.stl" scale="0.001 0.001 0.001"/>
-    </geometry>
-  </collision>
-</link>
-<link name="left_wheel">
-  <inertial>
-    <origin xyz="-4.6659614505450975e-09 0.009999959246660972 -3.8790217787854075e-08" rpy="0 0 0"/>
-    <mass value="0.17676171065422966"/>
-    <inertia ixx="0.00014" iyy="0.000267" izz="0.00014" ixy="0.0" iyz="0.0" ixz="-0.0"/>
-  </inertial>
-  <visual>
-    <origin xyz="-0.032937 -0.175618 -0.054935" rpy="0 0 0"/>
+    <origin xyz="-0.033069 -0.1761 -0.053887" rpy="0 0 0"/>
     <geometry>
       <mesh filename="package://wall_e_description/meshes/left_wheel_1.stl" scale="0.001 0.001 0.001"/>
     </geometry>
-    <material name="rubber_soft"/>
-  </visual>
-  <collision>
-    <origin xyz="-0.032937 -0.175618 -0.054935" rpy="0 0 0"/>
-    <geometry>
-      <mesh filename="package://wall_e_description/meshes/left_wheel_1.stl" scale="0.001 0.001 0.001"/>
-    </geometry>
-  </collision>
-</link>
-<link name="bin">
-  <inertial>
-    <origin xyz="0.022504658517767652 -0.00039207869774715576 0.17469334388419402" rpy="0 0 0"/>
+  </collision>
+</link>
+<link name="bin_1">
+  <inertial>
+    <origin xyz="-0.02250444308386567 0.00039161684009678815 0.17469329123226662" rpy="0 0 0"/>
     <mass value="12.102199401060787"/>
-    <inertia ixx="0.219187" iyy="0.186064" izz="0.190176" ixy="-0.000701" iyz="-0.000516" ixz="-0.000585"/>
-  </inertial>
-  <visual>
-    <origin xyz="-0.032937 -0.040618 -0.036435" rpy="0 0 0"/>
+    <inertia ixx="0.219187" iyy="0.186064" izz="0.190176" ixy="-0.000701" iyz="0.000516" ixz="0.000585"/>
+  </inertial>
+  <visual>
+    <origin xyz="-0.033069 -0.0411 -0.035387" rpy="0 0 0"/>
     <geometry>
       <mesh filename="package://wall_e_description/meshes/bin_1.stl" scale="0.001 0.001 0.001"/>
@@ -78,5 +78,5 @@
   </visual>
   <collision>
-    <origin xyz="-0.032937 -0.040618 -0.036435" rpy="0 0 0"/>
+    <origin xyz="-0.033069 -0.0411 -0.035387" rpy="0 0 0"/>
     <geometry>
       <mesh filename="package://wall_e_description/meshes/bin_1.stl" scale="0.001 0.001 0.001"/>
@@ -84,12 +84,12 @@
   </collision>
 </link>
-<link name="ydlidar_x4">
-  <inertial>
-    <origin xyz="-0.008294104236280672 -4.075333863429176e-08 0.03520110343257382" rpy="0 0 0"/>
+<link name="ydlidar_x4_1">
+  <inertial>
+    <origin xyz="0.012454197152355635 -4.2110431169861684e-07 0.03520105078064689" rpy="0 0 0"/>
     <mass value="1.1515616542314233"/>
-    <inertia ixx="0.000489" iyy="0.000861" izz="0.000987" ixy="-0.0" iyz="0.0" ixz="-0.000148"/>
-  </inertial>
-  <visual>
-    <origin xyz="-0.032937 -0.040618 -0.366435" rpy="0 0 0"/>
+    <inertia ixx="0.000489" iyy="0.000861" izz="0.000987" ixy="-0.0" iyz="0.0" ixz="0.000148"/>
+  </inertial>
+  <visual>
+    <origin xyz="-0.033069 -0.0411 -0.335387" rpy="0 0 0"/>
     <geometry>
       <mesh filename="package://wall_e_description/meshes/ydlidar_x4_1.stl" scale="0.001 0.001 0.001"/>
@@ -98,5 +98,5 @@
   </visual>
   <collision>
-    <origin xyz="-0.032937 -0.040618 -0.336435" rpy="0 0 0"/>
+    <origin xyz="-0.033069 -0.0411 -0.335387" rpy="0 0 0"/>
     <geometry>
       <mesh filename="package://wall_e_description/meshes/ydlidar_x4_1.stl" scale="0.001 0.001 0.001"/>
@@ -104,25 +104,106 @@
   </collision>
 </link>
+<link name="pan__1__1">
+  <inertial>
+    <origin xyz="0.04822559678907379 -0.11607817913674341 0.13061240970754556" rpy="0 0 0"/>
+    <mass value="3.94125611807655"/>
+    <inertia ixx="0.051476" iyy="0.025721" izz="0.03521" ixy="-8.7e-05" iyz="9.5e-05" ixz="-0.006231"/>
+  </inertial>
+  <visual>
+    <origin xyz="-0.164169 -0.157 -0.095987" rpy="0 0 0"/>
+    <geometry>
+      <mesh filename="package://wall_e_description/meshes/pan__1__1.stl" scale="0.001 0.001 0.001"/>
+    </geometry>
+    <material name="silver_default"/>
+  </visual>
+  <collision>
+    <origin xyz="-0.164169 -0.157 -0.095987" rpy="0 0 0"/>
+    <geometry>
+      <mesh filename="package://wall_e_description/meshes/pan__1__1.stl" scale="0.001 0.001 0.001"/>
+    </geometry>
+  </collision>
+</link>
+<link name="pan_left_arm_1">
+  <inertial>
+    <origin xyz="0.003000245244439148 -0.026606315345525516 0.11294972426483924" rpy="0 0 0"/>
+    <mass value="0.10558276566640609"/>
+    <inertia ixx="0.000719" iyy="0.000526" izz="0.000194" ixy="0.0" iyz="0.000294" ixz="0.0"/>
+  </inertial>
+  <visual>
+    <origin xyz="-0.168469 -0.171 -0.312605" rpy="0 0 0"/>
+    <geometry>
+      <mesh filename="package://wall_e_description/meshes/pan_left_arm_1.stl" scale="0.001 0.001 0.001"/>
+    </geometry>
+    <material name="steel_satin"/>
+  </visual>
+  <collision>
+    <origin xyz="-0.168469 -0.171 -0.312605" rpy="0 0 0"/>
+    <geometry>
+      <mesh filename="package://wall_e_description/meshes/pan_left_arm_1.stl" scale="0.001 0.001 0.001"/>
+    </geometry>
+  </collision>
+</link>
+<link name="pan_right_arm_1">
+  <inertial>
+    <origin xyz="0.003000194955287777 0.09335605146506651 0.06644584618966343" rpy="0 0 0"/>
+    <mass value="0.10558276566640609"/>
+    <inertia ixx="0.000719" iyy="9.9e-05" izz="0.00062" ixy="-0.0" iyz="-0.000215" ixz="-0.0"/>
+  </inertial>
+  <visual>
+    <origin xyz="-0.165969 0.09 -0.314825" rpy="0 0 0"/>
+    <geometry>
+      <mesh filename="package://wall_e_description/meshes/pan_right_arm_1.stl" scale="0.001 0.001 0.001"/>
+    </geometry>
+    <material name="steel_satin"/>
+  </visual>
+  <collision>
+    <origin xyz="-0.165969 0.09 -0.314825" rpy="0 0 0"/>
+    <geometry>
+      <mesh filename="package://wall_e_description/meshes/pan_right_arm_1.stl" scale="0.001 0.001 0.001"/>
+    </geometry>
+  </collision>
+</link>
 <joint name="left_drive" type="continuous">
-  <origin xyz="0.032937 -0.094382 0.054935" rpy="0 0 0"/>
+  <origin xyz="0.033069 -0.0939 0.053887" rpy="0 0 0"/>
   <parent link="base_link"/>
-  <child link="left_wheel"/>
-  <axis xyz="-0.0 1.0 0.0"/>
+  <child link="right_wheel_1"/>
+  <axis xyz="-0.0 -1.0 0.0"/>
 </joint>
 <joint name="right_drive" type="continuous">
-  <origin xyz="0.032937 0.175618 0.054935" rpy="0 0 0"/>
+  <origin xyz="0.033069 0.1761 0.053887" rpy="0 0 0"/>
   <parent link="base_link"/>
-  <child link="right_wheel"/>
+  <child link="left_wheel_1"/>
   <axis xyz="0.0 1.0 -0.0"/>
 </joint>
 <joint name="Rigid4" type="fixed">
-  <origin xyz="0.032937 0.040618 0.036435" rpy="0 0 0"/>
+  <origin xyz="0.033069 0.0411 0.035387" rpy="0 0 0"/>
   <parent link="base_link"/>
-  <child link="bin"/>
-</joint>
-<joint name="Rigid5" type="fixed">
-  <origin xyz="0.0 0.0 0.33" rpy="0 0 0"/>
-  <parent link="bin"/>
-  <child link="ydlidar_x4"/>
+  <child link="bin_1"/>
+</joint>
+<joint name="Rigid7" type="fixed">
+  <origin xyz="0.0 0.0 0.3" rpy="0 0 0"/>
+  <parent link="bin_1"/>
+  <child link="ydlidar_x4_1"/>
+</joint>
+<joint name="pan_joint" type="revolute">
+  <origin xyz="0.1311 0.1159 0.0606" rpy="0 0 0"/>
+  <parent link="bin_1"/>
+  <child link="pan__1__1"/>
+  <axis xyz="0.0 -1.0 0.0"/>
+  <limit upper="1.570796" lower="0.0" effort="100" velocity="100"/>
+</joint>
+<joint name="pan_left_arm" type="revolute">
+  <origin xyz="0.0043 0.014 0.216618" rpy="0 0 0"/>
+  <parent link="pan__1__1"/>
+  <child link="pan_left_arm_1"/>
+  <axis xyz="-1.0 -0.0 -0.0"/>
+  <limit upper="2.792527" lower="-0.785398" effort="100" velocity="100"/>
+</joint>
+<joint name="pan_right_arm" type="revolute">
+  <origin xyz="0.0018 -0.247 0.218838" rpy="0 0 0"/>
+  <parent link="pan__1__1"/>
+  <child link="pan_right_arm_1"/>
+  <axis xyz="-1.0 -0.0 -0.0"/>
+  <limit upper="0.087266" lower="-3.490659" effort="100" velocity="100"/>
 </joint>
 </robot>

Commit message: Add files via upload

File: wall_e_description/urdf/wall_e.xacro (robot description, xacro)
@@ -24,5 +24,5 @@
   </collision>
 </link>
-<link name="right_wheel_1">
+<link name="right_wheel">
   <inertial>
     <origin xyz="2.2009986355014943e-07 -0.010000421104311583 -9.144214505041326e-08" rpy="0 0 0"/>
@@ -44,5 +44,5 @@
   </collision>
 </link>
-<link name="left_wheel_1">
+<link name="left_wheel">
   <inertial>
     <origin xyz="2.2009986355014943e-07 0.009999578895688033 -9.144214514755777e-08" rpy="0 0 0"/>
@@ -64,5 +64,5 @@
   </collision>
 </link>
-<link name="bin_1">
+<link name="bin">
   <inertial>
     <origin xyz="-0.02250444308386567 0.00039161684009678815 0.17469329123226662" rpy="0 0 0"/>
@@ -84,5 +84,5 @@
   </collision>
 </link>
-<link name="ydlidar_x4_1">
+<link name="ydlidar_x4">
   <inertial>
     <origin xyz="0.012454197152355635 -4.2110431169861684e-07 0.03520105078064689" rpy="0 0 0"/>
@@ -91,18 +91,18 @@
   </inertial>
   <visual>
+    <origin xyz="-0.033069 -0.0411 -0.365387" rpy="0 0 0"/>
+    <geometry>
+      <mesh filename="package://wall_e_description/meshes/ydlidar_x4_1.stl" scale="0.001 0.001 0.001"/>
+    </geometry>
+    <material name="steel_satin"/>
+  </visual>
+  <collision>
     <origin xyz="-0.033069 -0.0411 -0.335387" rpy="0 0 0"/>
     <geometry>
       <mesh filename="package://wall_e_description/meshes/ydlidar_x4_1.stl" scale="0.001 0.001 0.001"/>
     </geometry>
-    <material name="steel_satin"/>
-  </visual>
-  <collision>
-    <origin xyz="-0.033069 -0.0411 -0.335387" rpy="0 0 0"/>
-    <geometry>
-      <mesh filename="package://wall_e_description/meshes/ydlidar_x4_1.stl" scale="0.001 0.001 0.001"/>
-    </geometry>
-  </collision>
-</link>
-<link name="pan__1__1">
+  </collision>
+</link>
+<link name="pan">
   <inertial>
     <origin xyz="0.04822559678907379 -0.11607817913674341 0.13061240970754556" rpy="0 0 0"/>
@@ -124,5 +124,5 @@
   </collision>
 </link>
-<link name="pan_left_arm_1">
+<link name="pan_left_arm">
   <inertial>
     <origin xyz="0.003000245244439148 -0.026606315345525516 0.11294972426483924" rpy="0 0 0"/>
@@ -144,5 +144,5 @@
   </collision>
 </link>
-<link name="pan_right_arm_1">
+<link name="pan_right_arm">
   <inertial>
     <origin xyz="0.003000194955287777 0.09335605146506651 0.06644584618966343" rpy="0 0 0"/>
@@ -164,14 +164,14 @@
   </collision>
 </link>
-<joint name="left_drive" type="continuous">
+<joint name="right_drive" type="continuous">
   <origin xyz="0.033069 -0.0939 0.053887" rpy="0 0 0"/>
   <parent link="base_link"/>
-  <child link="right_wheel_1"/>
-  <axis xyz="-0.0 -1.0 0.0"/>
-</joint>
-<joint name="right_drive" type="continuous">
+  <child link="right_wheel"/>
+  <axis xyz="-0.0 1.0 0.0"/>
+</joint>
+<joint name="left_drive" type="continuous">
   <origin xyz="0.033069 0.1761 0.053887" rpy="0 0 0"/>
   <parent link="base_link"/>
-  <child link="left_wheel_1"/>
+  <child link="left_wheel"/>
   <axis xyz="0.0 1.0 -0.0"/>
 </joint>
@@ -179,29 +179,29 @@
   <origin xyz="0.033069 0.0411 0.035387" rpy="0 0 0"/>
   <parent link="base_link"/>
-  <child link="bin_1"/>
+  <child link="bin"/>
 </joint>
 <joint name="Rigid7" type="fixed">
-  <origin xyz="0.0 0.0 0.3" rpy="0 0 0"/>
-  <parent link="bin_1"/>
-  <child link="ydlidar_x4_1"/>
+  <origin xyz="0.0 0.0 0.33" rpy="0 0 0"/>
+  <parent link="bin"/>
+  <child link="ydlidar_x4"/>
 </joint>
 <joint name="pan_joint" type="revolute">
   <origin xyz="0.1311 0.1159 0.0606" rpy="0 0 0"/>
-  <parent link="bin_1"/>
-  <child link="pan__1__1"/>
-  <axis xyz="0.0 -1.0 0.0"/>
-  <limit upper="1.570796" lower="0.0" effort="100" velocity="100"/>
-</joint>
-<joint name="pan_left_arm" type="revolute">
+  <parent link="bin"/>
+  <child link="pan"/>
+  <axis xyz="0.0 1.0 0.0"/>
+  <limit upper="1.570796" lower="0.0" effort="100" velocity="0.1"/>
+</joint>
+<joint name="left_arm" type="revolute">
   <origin xyz="0.0043 0.014 0.216618" rpy="0 0 0"/>
-  <parent link="pan__1__1"/>
-  <child link="pan_left_arm_1"/>
+  <parent link="pan"/>
+  <child link="pan_left_arm"/>
   <axis xyz="-1.0 -0.0 -0.0"/>
   <limit upper="2.792527" lower="-0.785398" effort="100" velocity="100"/>
 </joint>
-<joint name="pan_right_arm" type="revolute">
+<joint name="right_arm" type="revolute">
   <origin xyz="0.0018 -0.247 0.218838" rpy="0 0 0"/>
-  <parent link="pan__1__1"/>
-  <child link="pan_right_arm_1"/>
+  <parent link="pan"/>
+  <child link="pan_right_arm"/>
   <axis xyz="-1.0 -0.0 -0.0"/>
   <limit upper="0.087266" lower="-3.490659" effort="100" velocity="100"/>
